Commit message: Fix navigation environment and add grounding modules

File: romr_ros/urdf/romr_materials.xacro (robot description, xacro)
@@ -1,4 +1,4 @@
 <?xml version="1.0" ?>
-<robot name="romr_robot" xmlns:xacro="http://www.ros.org/wiki/xacro" >
+<robot name="romr_ros" xmlns:xacro="http://www.ros.org/wiki/xacro" >
 <material name="white">
   <color rgba="1 1 1 1"/>

File: romr_ros/urdf/romr_robot.xacro (robot description, xacro)
@@ -14,19 +14,16 @@
   </xacro:macro>
   <!-- ****************** Robot bases ***************************  -->
-  <!-- Define the center of the main robot chassis projected on the ground -->
-  <link name="base_footprint">
-    <xacro:footprint_inertia m="0" w="0" d="0" h="0"/>
-  </link>
-  <!-- The base footprint of the robot is located underneath the chassis -->
-  <joint name="base_joint" type="fixed">
-    <parent link="base_link"/>
-    <child link="base_footprint"/>
-    <origin xyz="0.0 0.0 -0.14" rpy="0 0 0"/>
-  </joint>
+  <!-- Define the center of the main robot chassis projected on the ground  -->
+  <link name="base_footprint"/>
+<joint name="base_joint" type="fixed">
+  <parent link="base_footprint"/>
+  <child link="base_link"/>
+  <origin xyz="0.0 0.0 0.14" rpy="0 0 0"/>
+</joint>
   <link name="base_link">
     <inertial>
-      <origin xyz="-0.0374777931065171 -0.000742607274570373 0.0517646177576365" rpy="0 0 0" />
-      <mass value="5.79174328389446" />
-      <inertia  ixx="0.0142969060262334" ixy="-4.92784367063061E-08" ixz="4.92627122966751E-05" iyy="0.0341323035296294" iyz="-2.71693609467846E-08" izz="0.0398544878636473" />
+      <origin xyz="-0.105449104749099 -6.2710990511583E-08 -0.0353826244627038" rpy="0 0 0" />
+      <mass value="5.62248188418557" />
+      <inertia ixx="0.0101780914316108" ixy="-7.67691385128644E-08" ixz="-4.89652321969437E-05" iyy="0.0274447769771713" iyz="2.47186505683292E-08" izz="0.0311711845501934" />
     </inertial>
     <visual>
@@ -41,18 +38,47 @@
       <origin xyz="0 0 0" rpy="0 0 0" />
       <geometry>
-        <mesh filename="package://romr_ros/meshes/base_link.STL" />
-      </geometry>
-    </collision>
-  </link>
+        <mesh
+          filename="package://romr_ros/meshes/base_link.STL" />
+      </geometry>
+    </collision>
+  </link>
+  <link name="leftwheel_link">
+    <inertial>
+      <origin xyz="5.55111512312578E-16 -0.0339035450394026 0"  rpy="0 0 0" />
+      <mass value="1.05822314366194" />
+      <inertia ixx="0.00185382833876821" ixy="-2.26580114666919E-17" ixz="5.78643446350551E-20" iyy="0.00311392342825296" iyz="-4.04063501773989E-19" izz="0.00185382833876821" />
+    </inertial>
+    <visual>
+      <origin xyz="0 0 0" rpy="0 0 0" />
+      <geometry>
+        <mesh filename="package://romr_ros/meshes/leftwheel_link.STL" />
+      </geometry>
+      <material name="black">
+      </material>
+    </visual>
+    <collision>
+      <origin xyz="0 0 0" rpy="0 0 0" />
+      <geometry>
+        <mesh filename="package://romr_ros/meshes/leftwheel_link.STL" />
+      </geometry>
+    </collision>
+  </link>
+  <joint name="leftwheel_joint" type="continuous">
+    <origin xyz="-0.019973 0.18486 -0.143" rpy="0 0 0" />
+    <parent link="base_link" />
+    <child link="leftwheel_link" />
+    <axis xyz="0 1 0" />
+    <limit effort="1" velocity="1" />
+  </joint>
   <link name="rightwheel_link">
     <inertial>
-      <origin xyz="-1.2143E-17 0.033904 1.3878E-17" rpy="0 0 0" />
-      <mass  value="1.0582" />
-      <inertia  ixx="0.0018538" ixy="-1.2518E-19" ixz="-7.2208E-20" iyy="0.0031139" iyz="1.5395E-18" izz="0.0018538" />
-    </inertial>
-    <visual>
-      <origin xyz="0 0 0" rpy="0 0 0" />
-      <geometry>
-        <mesh filename="package://romr_ros/meshes/rightwheel.STL" />
+      <origin xyz="0 0.0339035450394025 1.11022302462516E-16" rpy="0 0 0" />
+      <mass value="1.05822314366194" />
+      <inertia ixx="0.00185382833876821" ixy="-8.28317648396577E-19" ixz="-3.98214102856482E-20" iyy="0.00311392342825296" iyz="1.42645344260114E-18" izz="0.00185382833876821" />
+    </inertial>
+    <visual>
+      <origin xyz="0 0 0" rpy="0 0 0" />
+      <geometry>
+        <mesh filename="package://romr_ros/meshes/rightwheel_link.STL" />
       </geometry>
       <material name="black">
@@ -60,26 +86,54 @@
     </visual>
     <collision>
-      <origin xyz="0 0 0"  rpy="0 0 0" />
-      <geometry>
-        <mesh filename="package://romr_ros/meshes/rightwheel.STL" />
+      <origin xyz="0 0 0" rpy="0 0 0" />
+      <geometry>
+        <mesh filename="package://romr_ros/meshes/rightwheel_link.STL" />
       </geometry>
     </collision>
   </link>
   <joint name="rightwheel_joint" type="continuous">
-    <origin xyz="-0.12418 0.185 -0.063" rpy="0 0 3.1416" />
+    <origin xyz="-0.019973 -0.18514 -0.143" rpy="0 0 0" />
     <parent link="base_link" />
     <child link="rightwheel_link" />
     <axis xyz="0 1 0" />
-  </joint>
-  <link name="leftwheel_link">
-    <inertial>
-      <origin xyz="-2.4286E-17 -0.033904 4.1633E-17" rpy="0 0 0" />
-      <mass  value="1.0582" />
-      <inertia ixx="0.0018538" ixy="8.3854E-19" ixz="9.7745E-20" iyy="0.0031139" iyz="1.3019E-19" izz="0.0018538" />
-    </inertial>
-    <visual>
-      <origin xyz="0 0 0" rpy="0 0 0" />
-      <geometry>
-        <mesh filename="package://romr_ros/meshes/leftwheel.STL" />
+    <limit effort="1" velocity="1" />
+  </joint>
+  <link name="lidar_link">
+    <inertial>
+      <origin xyz="0.00295607523728636 0.000555575930936747 -0.0182096197435416" rpy="0 0 0" />
+      <mass value="0.165382751635991" />
+      <inertia ixx="7.87149168525185E-05" ixy="7.29372016034641E-07" ixz="2.13965886078915E-06" iyy="7.53405582518867E-05" iyz="4.42741020714694E-07" izz="0.000109946753058707" />
+    </inertial>
+    <visual>
+      <origin xyz="0 0 0" rpy="0 0 0" />
+      <geometry>
+        <mesh filename="package://romr_ros/meshes/lidar_link.STL" />
+      </geometry>
+      <material name="grey">
+      </material>
+    </visual>
+    <collision>
+      <origin xyz="0 0 0" rpy="0 0 0" />
+      <geometry>
+        <mesh filename="package://romr_ros/meshes/lidar_link.STL" />
+      </geometry>
+    </collision>
+  </link>
+  <joint name="lidar_joint" type="fixed">
+    <origin xyz="0.061574 -0.0034817 0.24851" rpy="0 0 0" />
+    <parent link="base_link" />
+    <child link="lidar_link" />
+    <axis xyz="0 0 0" />
+  </joint>
+  <link name="imu_link">
+    <inertial>
+      <origin xyz="0.0150149579003659 0.00012811592587525 0.000213690806863009"  rpy="0 0 0" />
+      <mass value="0.0515702797780248" />
+      <inertia ixx="1.57281367303655E-05" ixy="-1.2025506319508E-09" ixz="-1.58154472065039E-09" iyy="8.93790802791257E-06" iyz="2.18866082150114E-10" izz="1.43444156148991E-05" />
+    </inertial>
+    <visual>
+      <origin xyz="0 0 0" rpy="0 0 0" />
+      <geometry>
+        <mesh filename="package://romr_ros/meshes/imu_link.STL" />
       </geometry>
       <material name="black">
@@ -89,53 +143,55 @@
       <origin xyz="0 0 0" rpy="0 0 0" />
       <geometry>
-        <mesh filename="package://romr_ros/meshes/leftwheel.STL" />
-      </geometry>
-    </collision>
-  </link>
-  <joint name="leftwheel_joint" type="continuous">
-    <origin xyz="-0.12418 -0.185 -0.063" rpy="0 0 -3.1416" />
-    <parent link="base_link" />
-    <child link="leftwheel_link" />
+        <mesh filename="package://romr_ros/meshes/imu_link.STL" />
+      </geometry>
+    </collision>
+  </link>
+  <joint
+    name="imu_joint"
+    type="fixed">
+    <origin xyz="-0.19497 -0.011204 -0.023786" rpy="0 0 0" />
+    <parent link="base_link" />
+    <child link="imu_link" />
+    <axis xyz="0 0 0" />
+  </joint>
+  <link name="casterwheel_link">
+    <inertial>
+      <origin  xyz="-3.46944695195361E-18 0.015 -5.55111512312578E-17" rpy="0 0 0" />
+      <mass value="0.100245438847884" />
+      <inertia ixx="4.77227558263135E-05" ixy="-1.36719041040414E-20" ixz="-5.53311796152965E-21" iyy="8.67709468760967E-05" iyz="-1.33095397621866E-20" izz="4.77227558263135E-05" />
+    </inertial>
+    <visual>
+      <origin xyz="0 0 0" rpy="0 0 0" />
+      <geometry>
+        <mesh filename="package://romr_ros/meshes/casterwheel_link.STL" />
+      </geometry>
+      <material name="blue">
+      </material>
+    </visual>
+    <collision>
+      <origin xyz="0 0 0" rpy="0 0 0" />
+      <geometry>
+        <mesh filename="package://romr_ros/meshes/casterwheel_link.STL" />
+      </geometry>
+    </collision>
+  </link>
+  <joint name="casterwheel_joint" type="continuous">
+    <origin xyz="-0.39633 -0.013137 -0.1865" rpy="0 0 0" />
+    <parent link="base_link" />
+    <child link="casterwheel_link" />
     <axis xyz="0 1 0" />
   </joint>
-  <link name="casterwheel_link">
-    <inertial>
-      <origin xyz="-0.0032546 0.0053327 0.013127" rpy="0 0 0" />
-      <mass value="0.10255" />
-      <inertia ixx="9.4829E-05" ixy="-2.3412E-06" ixz="1.3145E-05" iyy="0.00012884" iyz="8.5135E-07" izz="5.2207E-05" />
-    </inertial>
-    <visual>
-      <origin xyz="0 0 0" rpy="0 0 0" />
-      <geometry>
-        <mesh filename="package://romr_ros/meshes/casterwheel.STL" />
-      </geometry>
-      <material name="blue">
-      </material>
-    </visual>
-    <collision>
-      <origin xyz="0 0 0" rpy="0 0 0" />
-      <geometry>
-        <mesh filename="package://romr_ros/meshes/casterwheel.STL" />
-      </geometry>
-    </collision>
-  </link>
-  <joint name="casterwheel_joint" type="fixed">
-    <origin xyz="0.25029 -0.01098 -0.1075" rpy="0 0 0" />
-    <parent link="base_link" />
-    <child link="casterwheel_link" />
-    <axis xyz="0 0 0" />
-  </joint>
-  <link name="lidar_link">
-    <inertial>
-      <origin xyz="0.00050486 -3.7855E-05 -0.025753" rpy="0 0 0" />
-      <mass  value="0.2064" />
-      <inertia ixx="0.00011156" ixy="-1.2701E-07" ixz="-1.6019E-06" iyy="0.00010988" iyz="1.201E-07" izz="0.0001391" />
-    </inertial>
-    <visual>
-      <origin xyz="0 0 0" rpy="0 0 0" />
-      <geometry>
-        <mesh filename="package://romr_ros/meshes/lidar.STL" />
-      </geometry>
-      <material name="grey">
+  <link name="camerat265_link">
+    <inertial>
+      <origin xyz="-0.00612660107785096 -3.85680560952839E-05 -1.90041413069553E-05"  rpy="0 0 0" />
+      <mass value="0.0309880995516971" />
+      <inertia ixx="3.02210611557782E-05" ixy="-1.65410508193904E-10" ixz="-4.89349387699645E-11" iyy="1.93627396026636E-06" iyz="-9.22648458352075E-11" izz="2.9001680210907E-05" />
+    </inertial>
+    <visual>
+      <origin xyz="0 0 0" rpy="0 0 0" />
+      <geometry>
+        <mesh filename="package://romr_ros/meshes/camerat265_link.STL" />
+      </geometry>
+      <material name="white">
       </material>
     </visual>
@@ -143,51 +199,24 @@
       <origin  xyz="0 0 0" rpy="0 0 0" />
       <geometry>
-        <mesh filename="package://romr_ros/meshes/lidar.STL" />
-      </geometry>
-    </collision>
-  </link>
-  <joint name="lidar_joint" type="fixed">
-    <origin xyz="0.00082049 0.00875 0.12332" rpy="0 0 0" />
-    <parent link="base_link" />
-    <child link="lidar_link" />
-    <axis xyz="0 0 1" />
-  </joint>
-  <link name="imu_link">
-    <inertial>
-      <origin xyz="-0.015015 -0.00012812 0.00021369" rpy="0 0 0" />
-      <mass value="0.05157" />
-      <inertia ixx="1.5728E-05" ixy="-1.2026E-09" ixz="1.5815E-09" iyy="8.9379E-06" iyz="-2.1887E-10" izz="1.4344E-05" />
-    </inertial>
-    <visual>
-      <origin xyz="0 0 0" rpy="0 0 0" />
-      <geometry>
-        <mesh filename="package://romr_ros/meshes/imu.STL" />
-      </geometry>
-      <material name="black">
-      </material>
-    </visual>
-    <collision>
-      <origin xyz="0 0 0" rpy="0 0 0" />
-      <geometry>
-        <mesh filename="package://romr_ros/meshes/imu.STL" />
-      </geometry>
-    </collision>
-  </link>
-  <joint name="imu_joint" type="fixed">
-    <origin xyz="0.05082 -0.0047896 0.053918" rpy="0 0 0" />
-    <parent link="base_link" />
-    <child link="imu_link" />
+        <mesh filename="package://romr_ros/meshes/camerat265_link.STL" />
+      </geometry>
+    </collision>
+  </link>
+  <joint name="camerat265_joint" type="fixed">
+    <origin xyz="0.057027 -0.07792 0.091015" rpy="0 0 0" />
+    <parent link="base_link" />
+    <child link="camerat265_link" />
     <axis xyz="0 0 0" />
   </joint>
   <link name="camerad435i_link">
     <inertial>
-      <origin xyz="0.0094812 3.7095E-05 -7.9734E-05" rpy="0 0 0" />
-      <mass value="0.032264" />
-      <inertia ixx="2.2098E-05" ixy="-1.4651E-10" ixz="2.902E-10" iyy="1.9467E-06" iyz="8.3417E-11" izz="2.1858E-05" />
-    </inertial>
-    <visual>
-      <origin xyz="0 0 0" rpy="0 0 0" />
-      <geometry>
-        <mesh filename="package://romr_ros/meshes/camerad435i.STL" />
+      <origin xyz="-0.00948120491609372 -3.70946771987568E-05 -7.97343604980183E-05" rpy="0 0 0" />
+      <mass value="0.0322638693424906" />
+      <inertia ixx="2.20979298020458E-05" ixy="-1.46511332900792E-10" ixz="-2.90204280421224E-10" iyy="1.94666557711069E-06" iyz="-8.34172635681561E-11" izz="2.18579669241807E-05" />
+    </inertial>
+    <visual>
+      <origin xyz="0 0 0" rpy="0 0 0" />
+      <geometry>
+        <mesh filename="package://romr_ros/meshes/camerad435i_link.STL" />
       </geometry>
       <material name="white">
@@ -195,42 +224,24 @@
     </visual>
     <collision>
-      <origin xyz="0 0 0" rpy="0 0 0" />
-      <geometry>
-        <mesh filename="package://romr_ros/meshes/camerad435i.STL" />
+      <origin  xyz="0 0 0" rpy="0 0 0" />
+      <geometry>
+        <mesh filename="package://romr_ros/meshes/camerad435i_link.STL" />
       </geometry>
     </collision>
   </link>
   <joint name="camerad435i_joint" type="fixed">
-    <origin xyz="-0.20718 -0.08268 0.17016" rpy="0 0 0" />
-    <parent  link="base_link" />
+    <origin xyz="0.063027 0.085996 0.087815" rpy="0 0 0" />
+    <parent link="base_link" />
     <child link="camerad435i_link" />
     <axis xyz="0 0 0" />
   </joint>
-  <link name="camerat265_link">
-    <inertial>
-      <origin xyz="0.0061266 3.8568E-05 -1.9004E-05" rpy="0 0 0" />
-      <mass value="0.030988" />
-      <inertia ixx="3.0221E-05" ixy="-1.6541E-10" ixz="4.8935E-11" iyy="1.9363E-06" iyz="9.2265E-11" izz="2.9002E-05" />
-    </inertial>
-    <visual>
-      <origin  xyz="0 0 0"  rpy="0 0 0" />
-      <geometry>
-        <mesh filename="package://romr_ros/meshes/camerat265.STL" />
-      </geometry>
-      <material name="white">
-      </material>
-    </visual>
-    <collision>
-      <origin xyz="0 0 0" rpy="0 0 0" />
-      <geometry>
-        <mesh filename="package://romr_ros/meshes/camerat265.STL" />
-      </geometry>
-    </collision>
-  </link>
-  <joint name="camerat265_joint" type="fixed">
-    <origin  xyz="-0.20118 0.080908 0.16952" rpy="0 0 0" />
-    <parent link="base_link" />
-    <child link="camerat265_link" />
-    <axis xyz="0 0 0" />
+  <link name="camera_rgbd_frame">
+  <origin xyz="0 0 0" rpy="0 0 0"/>
+  </link>
+  <joint name="camera_rgbd_frame_joint" type="fixed">
+    <origin xyz="0.057027 -0.07792 0.091015" rpy="0 0 0" />
+    <!--origin xyz="0 0 0" rpy="0 0 1.5707"/-->
+    <parent link="base_link"/>
+    <child link="camera_rgbd_frame"/>
   </joint>
 </robot>
